Commit message: Initial commit

File: antonie_description/urdf/antonie.urdf (robot description, URDF)
Before this commit: robot three_joint_gripper, 5 links, 4 joints
Links:
- removed link world
- removed link wrist_mount
- added link base_link; collision cylinder length=0.6 radius=0.2; visual cylinder length=0.6 radius=0.2
- added link link_1; collision cylinder length=0.5 radius=0.1; visual cylinder length=0.5 radius=0.1
- added link link_2; collision cylinder length=0.5 radius=0.08; visual cylinder length=0.5 radius=0.08
- added link link_3; collision cylinder length=0.4 radius=0.06; visual cylinder length=0.4 radius=0.06
- link gripper_base: geometry collision box size=0.2 0.05 0.05; visual box size=0.2 0.05 0.05
- link left_finger: geometry collision box size=0.02 0.02 0.1; visual box size=0.02 0.02 0.1
- link right_finger: geometry collision box size=0.02 0.02 0.1; visual box size=0.02 0.02 0.1
Joints:
- removed joint left_finger_joint
- removed joint right_finger_joint
- removed joint world_to_base
- removed joint wrist_roll_joint
- added joint arm_0_joint: type revolute, parent base_link, child link_1, origin xyz=0 0 0.3, axis 0 0 1, limit lower=-3.14 upper=3.14 effort=10 velocity=1.0
- added joint arm_1_joint: type revolute, parent link_1, child link_2, origin xyz=0 0 0.5, axis 0 1 0, limit lower=-1.57 upper=1.57 effort=10 velocity=1.0
- added joint arm_2_joint: type revolute, parent link_2, child link_3, origin xyz=0 0 0.5, axis 0 1 0, limit lower=-1.57 upper=1.57 effort=10 velocity=1.0
- added joint gripper_1_joint: type prismatic, parent gripper_base, child left_finger, origin xyz=-0.08 0 0, axis 1 0 0, limit lower=0.0 upper=0.05 effort=5 velocity=0.5
- added joint gripper_2_joint: type prismatic, parent gripper_base, child right_finger, origin xyz=0.08 0 0, axis -1 0 0, limit lower=0.0 upper=0.05 effort=5 velocity=0.5
- added joint gripper_fixed_joint: type fixed, parent link_3, child gripper_base, origin xyz=0 0 0.4 rpy=0 0 0
